File: planetarium/seiza_ittose/seiza_ittose/seiza_ittose.kicad_sch (KiCad schematic)
At the start: 28 parts, among them J1 Jack-DC, J10 Jack-DC, J11 Jack-DC, J12 Jack-DC, J13 Jack-DC, J2 Jack-DC, J3 Jack-DC, J4 Jack-DC, J5 Jack-DC, J6 Jack-DC, J7 Jack-DC, J8 Jack-DC, J9 Jack-DC, Q1 NP52N06SLG, Q2 NP52N06SLG, Q3 NP52N06SLG, Q4 NP52N06SLG, Q5 NP52N06SLG, Q6 NP52N06SLG, Q7 NP52N06SLG, Q8 NP52N06SLG, Q9 NP52N06SLG, U1 XIAO-ESP32-C3-SMD

Commit message: chore
Parts:
- D1: footprint (none) -> GS1010FL:GS1010FL
Other:
- note added: "要検討 アンテナの位置"
- note removed: "TO DO: ダイオードの実装のみ"
Changed lines of the file:
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@@
 	(generator_version "9.0")
 	(paper "A4")
-	(text "TO DO: ダイオードの実装のみ"
+	(text "要検討　アンテナの位置"
 		(exclude_from_sim no)
-		(at 231.648 153.67 0)
+		(at 224.028 150.368 0)
 		(effects
 			(font
@@
 			)
 		)
-		(property "Footprint" ""
+		(property "Footprint" "GS1010FL:GS1010FL"
 			(at 250.19 95.25 0)
 			(effects
